File: PCBs/Roaster Breakout/Roaster Breakout.brd (EAGLE design)
At the start: 48.8 x 39.6 mm, 9 parts

Commit message: site updates and pcb labeling
Other:
- board size 48.8 x 39.6 mm -> 52.4 x 42.4 mm
- board text added: "FAN CTRL"
